File: board/core.sch (KiCad schematic (older format))
At the start: 3 parts

Commit message: WIP
Parts:
- added J?: JTAG, symbol Connector_Generic:Conn_02x05_Odd_Even
- added RN?: 4.7k, Resistor_THT:R_Array_SIP5, symbol Device:R_Network04
- added U?: 74AC573, symbol 74xx:74LS574
Connections:
- net labels added: A19, A20, A21, A22, A23, IO6SELB, ~IO5SELB
- net labels removed: BA0, BA1, BA2, BA3, BA4, BA5, BA6, BA7, RESET
- wire segments 129 -> 158
- no-connect marks 3 -> 6
Other:
- moved on the sheet: U?
