File: board/uart.sch (KiCad schematic (older format))
At the start: 18 parts, among them U10 MAX238, U11 MAX238, U8 3.6864M, U9 SC28L92

Commit message: RC1 of schematic and initial board layout
Parts:
- C27: renamed from C9; value 1u -> 0.1u; footprint (none) -> Capacitor_THT:C_Rect_L4.6mm_W2.0mm_P2.50mm_MKS02_FKP02
- C28: renamed from C10; value 1u -> 0.1u; footprint (none) -> Capacitor_THT:C_Rect_L4.6mm_W2.0mm_P2.50mm_MKS02_FKP02
- C29: renamed from C11; value 1u -> 0.1u; footprint (none) -> Capacitor_THT:C_Rect_L4.6mm_W2.0mm_P2.50mm_MKS02_FKP02
- C30: renamed from C12; value 1u -> 0.1u; footprint (none) -> Capacitor_THT:C_Rect_L4.6mm_W2.0mm_P2.50mm_MKS02_FKP02
- C31: renamed from C13; footprint (none) -> Capacitor_THT:CP_Radial_D5.0mm_P2.00mm
- C32: renamed from C14; footprint (none) -> Capacitor_THT:CP_Radial_D5.0mm_P2.00mm
- C33: renamed from C15; footprint (none) -> Capacitor_THT:CP_Radial_D5.0mm_P2.00mm
- C34: renamed from C16; footprint (none) -> Capacitor_THT:CP_Radial_D5.0mm_P2.00mm
- C35: renamed from C17; footprint (none) -> Capacitor_THT:CP_Radial_D5.0mm_P2.00mm
- C36: renamed from C18; footprint (none) -> Capacitor_THT:CP_Radial_D5.0mm_P2.00mm
- C37: renamed from C19; footprint (none) -> Capacitor_THT:CP_Radial_D5.0mm_P2.00mm
- C38: renamed from C20; footprint (none) -> Capacitor_THT:CP_Radial_D5.0mm_P2.00mm
- C39: renamed from C21; footprint (none) -> Capacitor_THT:CP_Radial_D5.0mm_P2.00mm
- C40: renamed from C22; footprint (none) -> Capacitor_THT:CP_Radial_D5.0mm_P2.00mm
- U12: renamed from U8; footprint (none) -> Package_DIP:DIP-8_W7.62mm_Socket
- U14: renamed from U10; footprint (none) -> Package_DIP:DIP-24_W7.62mm_Socket
- U15: renamed from U11; footprint (none) -> Package_DIP:DIP-24_W7.62mm_Socket
- renumbered U9 to U13

Commit message: RC1 of schematic and initial board layout
Parts:
- renumbered C27 to C21, C28 to C22, C29 to C23, C30 to C24, C31 to C25, C32 to C26, C33 to C27, C34 to C28, C35 to C29, C36 to C30, C37 to C31, C38 to C32, C39 to C33, C40 to C34
Changed lines of the file:
@@
 AR Path="/61B43476/6208E351" Ref="#PWR?"  Part="1"
 AR Path="/62053143/6208E351" Ref="#PWR?"  Part="1"
-AR Path="/62053498/6208E351" Ref="#PWR080"  Part="1"
-F 0 "#PWR080" H 3400 5000 50  0001 C CNN
+AR Path="/62053498/6208E351" Ref="#PWR074"  Part="1"
+F 0 "#PWR074" H 3400 5000 50  0001 C CNN
 F 1 "GND" H 3405 5077 50  0000 C CNN
 F 2 "" H 3400 5250 50  0001 C CNN
@@
 AR Path="/61B43476/620909CF" Ref="#PWR?"  Part="1"
 AR Path="/62053143/620909CF" Ref="#PWR?"  Part="1"
-AR Path="/62053498/620909CF" Ref="#PWR079"  Part="1"
-F 0 "#PWR079" H 3400 1800 50  0001 C CNN
+AR Path="/62053498/620909CF" Ref="#PWR073"  Part="1"
+F 0 "#PWR073" H 3400 1800 50  0001 C CNN
 F 1 "+5V" H 3415 2123 50  0000 C CNN
 F 2 "" H 3400 1950 50  0001 C CNN
@@
 AR Path="/61B43476/620A9003" Ref="#PWR?"  Part="1"
 AR Path="/62053143/620A9003" Ref="#PWR?"  Part="1"
-AR Path="/62053498/620A9003" Ref="#PWR077"  Part="1"
-F 0 "#PWR077" H 1550 4850 50  0001 C CNN
+AR Path="/62053498/620A9003" Ref="#PWR071"  Part="1"
+F 0 "#PWR071" H 1550 4850 50  0001 C CNN
 F 1 "GND" H 1555 4927 50  0000 C CNN
 F 2 "" H 1550 5100 50  0001 C CNN
@@
 AR Path="/61B43476/620AAA2E" Ref="#PWR?"  Part="1"
 AR Path="/62053143/620AAA2E" Ref="#PWR?"  Part="1"
-AR Path="/62053498/620AAA2E" Ref="#PWR076"  Part="1"
-F 0 "#PWR076" H 1550 3700 50  0001 C CNN
+AR Path="/62053498/620AAA2E" Ref="#PWR070"  Part="1"
+F 0 "#PWR070" H 1550 3700 50  0001 C CNN
 F 1 "+5V" H 1565 4023 50  0000 C CNN
 F 2 "" H 1550 3850 50  0001 C CNN
@@
 AR Path="/60EE1618/620B1487" Ref="#PWR?"  Part="1"
 AR Path="/61ADDFAC/620B1487" Ref="#PWR?"  Part="1"
-AR Path="/62053498/620B1487" Ref="#PWR078"  Part="1"
-F 0 "#PWR078" H 1700 7350 50  0001 C CNN
+AR Path="/62053498/620B1487" Ref="#PWR072"  Part="1"
+F 0 "#PWR072" H 1700 7350 50  0001 C CNN
 F 1 "GND" H 1705 7427 50  0000 C CNN
 F 2 "" H 1700 7600 50  0001 C CNN
@@
 AR Path="/60EE1618/620B148D" Ref="C?"  Part="1"
 AR Path="/61ADDFAC/620B148D" Ref="C?"  Part="1"
-AR Path="/62053498/620B148D" Ref="C27"  Part="1"
-F 0 "C27" H 1042 7346 50  0001 L CNN
+AR Path="/62053498/620B148D" Ref="C21"  Part="1"
+F 0 "C21" H 1042 7346 50  0001 L CNN
 F 1 "0.1u" H 1042 7300 50  0001 L CNN
 F 2 "Capacitor_THT:C_Rect_L4.6mm_W2.0mm_P2.50mm_MKS02_FKP02" H 950 7300 50  0001 C CNN
@@
 AR Path="/60EE1618/620B1493" Ref="#PWR?"  Part="1"
 AR Path="/61ADDFAC/620B1493" Ref="#PWR?"  Part="1"
-AR Path="/62053498/620B1493" Ref="#PWR075"  Part="1"
-F 0 "#PWR075" H 950 6850 50  0001 C CNN
+AR Path="/62053498/620B1493" Ref="#PWR069"  Part="1"
+F 0 "#PWR069" H 950 6850 50  0001 C CNN
 F 1 "+5V" H 965 7173 50  0000 C CNN
 F 2 "" H 950 7000 50  0001 C CNN
@@
 AR Path="/60EE1618/620B149F" Ref="C?"  Part="1"
 AR Path="/61ADDFAC/620B149F" Ref="C?"  Part="1"
-AR Path="/62053498/620B149F" Ref="C28"  Part="1"
-F 0 "C28" H 1292 7346 50  0001 L CNN
+AR Path="/62053498/620B149F" Ref="C22"  Part="1"
+F 0 "C22" H 1292 7346 50  0001 L CNN
 F 1 "0.1u" H 1292 7300 50  0001 L CNN
 F 2 "Capacitor_THT:C_Rect_L4.6mm_W2.0mm_P2.50mm_MKS02_FKP02" H 1200 7300 50  0001 C CNN
@@
 AR Path="/61B43476/62A44A61" Ref="#PWR?"  Part="1"
 AR Path="/62053143/62A44A61" Ref="#PWR?"  Part="1"
-AR Path="/62053498/62A44A61" Ref="#PWR081"  Part="1"
-F 0 "#PWR081" H 7950 650 50  0001 C CNN
+AR Path="/62053498/62A44A61" Ref="#PWR075"  Part="1"
+F 0 "#PWR075" H 7950 650 50  0001 C CNN
 F 1 "+5V" H 7965 973 50  0000 C CNN
 F 2 "" H 7950 800 50  0001 C CNN
@@
 AR Path="/61B43476/62A847D6" Ref="#PWR?"  Part="1"
 AR Path="/62053143/62A847D6" Ref="#PWR?"  Part="1"
-AR Path="/62053498/62A847D6" Ref="#PWR082"  Part="1"
-F 0 "#PWR082" H 7950 3100 50  0001 C CNN
+AR Path="/62053498/62A847D6" Ref="#PWR076"  Part="1"
+F 0 "#PWR076" H 7950 3100 50  0001 C CNN
 F 1 "GND" H 7955 3177 50  0000 C CNN
 F 2 "" H 7950 3350 50  0001 C CNN
@@
 	7950 2950 7950 3150
 $Comp
-L Device:CP_Small C31
+L Device:CP_Small C25
 U 1 1 62A89389
 P 6600 1500
-F 0 "C31" H 6688 1546 50  0000 L CNN
+F 0 "C25" H 6688 1546 50  0000 L CNN
 F 1 "1.0u" H 6688 1455 50  0000 L CNN
 F 2 "Capacitor_THT:CP_Radial_D5.0mm_P2.00mm" H 6600 1500 50  0001 C CNN
@@
 	7000 1450 7450 1450
 $Comp
-L Device:CP_Small C38
+L Device:CP_Small C32
 U 1 1 62AA1EFF
 P 8650 2950
-F 0 "C38" H 8562 2904 50  0000 R CNN
+F 0 "C32" H 8562 2904 50  0000 R CNN
 F 1 "1.0u" H 8562 2995 50  0000 R CNN
 F 2 "Capacitor_THT:CP_Radial_D5.0mm_P2.00mm" H 8650 2950 50  0001 C CNN
@@
 $EndComp
 $Comp
-L Device:CP_Small C37
+L Device:CP_Small C31
 U 1 1 62AA3338
 P 8650 1200
-F 0 "C37" H 8738 1246 50  0000 L CNN
+F 0 "C31" H 8738 1246 50  0000 L CNN
 F 1 "1.0u" H 8738 1155 50  0000 L CNN
 F 2 "Capacitor_THT:CP_Radial_D5.0mm_P2.00mm" H 8650 1200 50  0001 C CNN
@@
 	7950 3150 7950 3350
 $Comp
-L Device:CP_Small C35
+L Device:CP_Small C29
 U 1 1 62B0A85A
 P 7400 1000
-F 0 "C35" V 7300 950 50  0000 L CNN
+F 0 "C29" V 7300 950 50  0000 L CNN
 F 1 "1.0u" V 7500 900 50  0000 L CNN
 F 2 "Capacitor_THT:CP_Radial_D5.0mm_P2.00mm" H 7400 1000 50  0001 C CNN
@@
 	6600 1600 7000 1600
 $Comp
-L Device:CP_Small C32
+L Device:CP_Small C26
 U 1 1 62BB9E2D
 P 6600 2800
-F 0 "C32" H 6688 2846 50  0000 L CNN
+F 0 "C26" H 6688 2846 50  0000 L CNN
 F 1 "1.0u" H 6688 2755 50  0000 L CNN
 F 2 "Capacitor_THT:CP_Radial_D5.0mm_P2.00mm" H 6600 2800 50  0001 C CNN
@@
 AR Path="/61B43476/62BD5752" Ref="#PWR?"  Part="1"
 AR Path="/62053143/62BD5752" Ref="#PWR?"  Part="1"
-AR Path="/62053498/62BD5752" Ref="#PWR083"  Part="1"
-F 0 "#PWR083" H 7950 3700 50  0001 C CNN
+AR Path="/62053498/62BD5752" Ref="#PWR077"  Part="1"
+F 0 "#PWR077" H 7950 3700 50  0001 C CNN
 F 1 "+5V" H 7965 4023 50  0000 C CNN
 F 2 "" H 7950 3850 50  0001 C CNN
@@
 AR Path="/61B43476/62BD5766" Ref="#PWR?"  Part="1"
 AR Path="/62053143/62BD5766" Ref="#PWR?"  Part="1"
-AR Path="/62053498/62BD5766" Ref="#PWR084"  Part="1"
-F 0 "#PWR084" H 7950 6150 50  0001 C CNN
+AR Path="/62053498/62BD5766" Ref="#PWR078"  Part="1"
+F 0 "#PWR078" H 7950 6150 50  0001 C CNN
 F 1 "GND" H 7955 6227 50  0000 C CNN
 F 2 "" H 7950 6400 50  0001 C CNN
@@
 	7950 6000 7950 6200
 $Comp
-L Device:CP_Small C33
+L Device:CP_Small C27
 U 1 1 62BD576D
 P 6600 4550
-F 0 "C33" H 6688 4596 50  0000 L CNN
+F 0 "C27" H 6688 4596 50  0000 L CNN
 F 1 "1.0u" H 6688 4505 50  0000 L CNN
 F 2 "Capacitor_THT:CP_Radial_D5.0mm_P2.00mm" H 6600 4550 50  0001 C CNN
@@
 	7000 4500 7450 4500
 $Comp
-L Device:CP_Small C40
+L Device:CP_Small C34
 U 1 1 62BD5777
 P 8650 6000
-F 0 "C40" H 8562 5954 50  0000 R CNN
+F 0 "C34" H 8562 5954 50  0000 R CNN
 F 1 "1.0u" H 8562 6045 50  0000 R CNN
 F 2 "Capacitor_THT:CP_Radial_D5.0mm_P2.00mm" H 8650 6000 50  0001 C CNN
@@
 $EndComp
 $Comp
-L Device:CP_Small C39
+L Device:CP_Small C33
 U 1 1 62BD577D
 P 8650 4250
-F 0 "C39" H 8738 4296 50  0000 L CNN
+F 0 "C33" H 8738 4296 50  0000 L CNN
 F 1 "1.0u" H 8738 4205 50  0000 L CNN
 F 2 "Capacitor_THT:CP_Radial_D5.0mm_P2.00mm" H 8650 4250 50  0001 C CNN
@@
 	7950 6200 7950 6400
 $Comp
-L Device:CP_Small C36
+L Device:CP_Small C30
 U 1 1 62BD579C
 P 7400 4050
-F 0 "C36" V 7300 4000 50  0000 L CNN
+F 0 "C30" V 7300 4000 50  0000 L CNN
 F 1 "1.0u" V 7500 3950 50  0000 L CNN
 F 2 "Capacitor_THT:CP_Radial_D5.0mm_P2.00mm" H 7400 4050 50  0001 C CNN
@@
 	6600 4650 7000 4650
 $Comp
-L Device:CP_Small C34
+L Device:CP_Small C28
 U 1 1 62BD57C1
 P 6600 5850
-F 0 "C34" H 6688 5896 50  0000 L CNN
+F 0 "C28" H 6688 5896 50  0000 L CNN
 F 1 "1.0u" H 6688 5805 50  0000 L CNN
 F 2 "Capacitor_THT:CP_Radial_D5.0mm_P2.00mm" H 6600 5850 50  0001 C CNN
@@
 AR Path="/60EE1618/61FE1F40" Ref="C?"  Part="1"
 AR Path="/61ADDFAC/61FE1F40" Ref="C?"  Part="1"
-AR Path="/62053498/61FE1F40" Ref="C29"  Part="1"
-F 0 "C29" H 1542 7346 50  0001 L CNN
+AR Path="/62053498/61FE1F40" Ref="C23"  Part="1"
+F 0 "C23" H 1542 7346 50  0001 L CNN
 F 1 "0.1u" H 1542 7300 50  0001 L CNN
 F 2 "Capacitor_THT:C_Rect_L4.6mm_W2.0mm_P2.50mm_MKS02_FKP02" H 1450 7300 50  0001 C CNN
@@
 AR Path="/60EE1618/61FE1F46" Ref="C?"  Part="1"
 AR Path="/61ADDFAC/61FE1F46" Ref="C?"  Part="1"
-AR Path="/62053498/61FE1F46" Ref="C30"  Part="1"
-F 0 "C30" H 1792 7346 50  0001 L CNN
+AR Path="/62053498/61FE1F46" Ref="C24"  Part="1"
+F 0 "C24" H 1792 7346 50  0001 L CNN
 F 1 "0.1u" H 1792 7300 50  0001 L CNN
 F 2 "Capacitor_THT:C_Rect_L4.6mm_W2.0mm_P2.50mm_MKS02_FKP02" H 1700 7300 50  0001 C CNN
