File: board/cpu.sch (KiCad schematic (older format))
At the start: 15 parts, among them U1 74HC21, U2 W65C816SxPL, U3 74ACT245, U4 74AC573, U5 74ACT245, U6 74ACT245

Commit message: RC1 of schematic and initial board layout
Parts:
- removed C6, C7: 1u, symbol Device:C_Small
- removed U5, U6: 74ACT245, symbol 74xx:74HC245
- C12: renamed from C1; value 1u -> 0.1u; footprint (none) -> Capacitor_THT:C_Rect_L4.6mm_W2.0mm_P2.50mm_MKS02_FKP02
- C13: renamed from C2; value 1u -> 0.1u; footprint (none) -> Capacitor_THT:C_Rect_L4.6mm_W2.0mm_P2.50mm_MKS02_FKP02
- C14: renamed from C3; value 1u -> 0.1u; footprint (none) -> Capacitor_THT:C_Rect_L4.6mm_W2.0mm_P2.50mm_MKS02_FKP02
- C15: renamed from C4; value 1u -> 0.1u; footprint (none) -> Capacitor_THT:C_Rect_L4.6mm_W2.0mm_P2.50mm_MKS02_FKP02
- C16: renamed from C5; value 1u -> 0.1u; footprint (none) -> Capacitor_THT:C_Rect_L4.6mm_W2.0mm_P2.50mm_MKS02_FKP02
- U6: renamed from U1; value 74HC21 -> SN74HC21N; footprint (none) -> Package_DIP:DIP-14_W7.62mm_Socket
- U7: renamed from U2; footprint (none) -> Package_LCC:PLCC-44_THT-Socket
- U8: renamed from U3; value 74ACT245 -> SN74AHCT245N; footprint (none) -> Package_DIP:DIP-20_W7.62mm_Socket
- U9: renamed from U4; value 74AC573 -> SN74AC573N; footprint (none) -> Package_DIP:DIP-20_W7.62mm_Socket
Other:
- moved on the sheet: RN1, RN2, U6A, U6B, U6C, U7, U8, U9

Commit message: Fix footprint for RESET and NMI button handlers Fix symbol for '573 latch
Parts:
- U9: value SN74AC573N -> SN74AHC573N; symbol 74xx:74LS574 -> 74xx:74LS573
Changed lines of the file:
@@
 Connection ~ 5800 6900
 $Comp
-L 74xx:74LS574 U9
+L 74xx:74LS573 U9
 U 1 1 61595EA3
 P 5800 6100
 F 0 "U9" H 5550 6750 50  0000 C CNN
-F 1 "SN74AC573N" H 6100 6750 50  0000 C CNN
+F 1 "SN74AHC573N" H 6100 6750 50  0000 C CNN
 F 2 "Package_DIP:DIP-20_W7.62mm_Socket" H 5800 6100 50  0001 C CNN
 F 3 "" H 5800 6100 50  0001 C CNN
