File: board/ports.sch (KiCad schematic (older format))
At the start: 24 parts, among them J1 USER PORT, J10 SLOT 3, J11 NMI SWITCH, J2 SERIAL A, J3 SERIAL B, J4 SD CARD, J5 DC IN 5V, J6 SLOT 1, J7 JTAG, J8 SLOT 2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

Commit message: RC1 of schematic and initial board layout
Parts:
- removed J11: NMI SWITCH, symbol Connector_Generic:Conn_01x02
- removed J9: RESET SWITCH, symbol Connector_Generic:Conn_01x02
- added SW1, SW2: SW_Push, Button_Switch_THT:SW_PUSH_6mm_H5mm, symbol Switch:SW_Push
- C17: renamed from C28; value 1u -> 0.1u; footprint (none) -> Capacitor_THT:C_Rect_L4.6mm_W2.0mm_P2.50mm_MKS02_FKP02
- C18: renamed from C29; value 1u -> 0.1u; footprint (none) -> Capacitor_THT:C_Rect_L4.6mm_W2.0mm_P2.50mm_MKS02_FKP02
- C19: renamed from C30; footprint (none) -> Capacitor_THT:C_Rect_L4.6mm_W2.0mm_P2.50mm_MKS02_FKP02
- C20: renamed from C31; footprint (none) -> Capacitor_THT:CP_Radial_D5.0mm_P2.00mm
- C21: renamed from C32; footprint (none) -> Capacitor_THT:CP_Radial_D5.0mm_P2.00mm
- C22: renamed from C33; footprint (none) -> Capacitor_THT:C_Rect_L4.6mm_W2.0mm_P2.50mm_MKS02_FKP02
- C23: renamed from C34; footprint (none) -> Capacitor_THT:C_Rect_L4.6mm_W2.0mm_P2.50mm_MKS02_FKP02
- C24: renamed from C35; footprint (none) -> Capacitor_THT:CP_Radial_D5.0mm_P2.00mm
- C25: renamed from C36; footprint (none) -> Capacitor_THT:C_Rect_L4.6mm_W2.0mm_P2.50mm_MKS02_FKP02
- C26: renamed from C37; footprint (none) -> Capacitor_THT:CP_Radial_D5.0mm_P2.00mm
- J1: footprint (none) -> Connector_PinHeader_1.00mm:PinHeader_2x17_P1.00mm_Vertical
- J2, J3: footprint (none) -> Connector_Dsub:DSUB-9_Male_Horizontal_P2.77x2.84mm_EdgePinOffset4.94mm_Housed_MountingHolesOffset7.48mm
- J4: footprint (none) -> Connector_PinHeader_2.54mm:PinHeader_1x06_P2.54mm_Vertical
- J5: footprint (none) -> Connector_BarrelJack:BarrelJack_Horizontal
- J6, J8: footprint (none) -> Connector_Samtec_HLE_THT:Samtec_HLE-120-02-xx-DV-TE_2x20_P2.54mm_Horizontal
- J7: footprint (none) -> Connector_IDC:IDC-Header_2x05_P2.54mm_Vertical
- J9: renamed from J10; footprint (none) -> Connector_Samtec_HLE_THT:Samtec_HLE-120-02-xx-DV-TE_2x20_P2.54mm_Horizontal
- U10: renamed from U17; footprint Package_TO_SOT_SMD:SOT-23 -> jrc:TO-92_reverse
- U11: renamed from U18; footprint Package_TO_SOT_SMD:SOT-23 -> jrc:TO-92_reverse
Connections:
- net GND: now also SW1.1, SW2.1
- net NMIB: now also SW2.2
- net PHI2: no longer J6.12 (Φ2), J8.12 (Φ2)
- net RDB: no longer J6.14 (~RD), J8.14 (~RD)
- net RESETB: now also SW1.2
- net RWB: no longer J6.13 (R/~W), J8.13 (R/~W)
- net WRB: no longer J6.15 (~WR), J8.15 (~WR)
- new net XPHI2: J6.12 (Φ2), J8.12 (Φ2)
- new net XRDB: J6.14 (~RD), J8.14 (~RD)
- new net XRWB: J6.13 (R/~W), J8.13 (R/~W)
- new net XWRB: J6.15 (~WR), J8.15 (~WR)

Commit message: Use custom footprint for slots to get more favorable pin numbering for layout purposes.
Parts:
- J6, J8, J9: footprint Connector_Samtec_HLE_THT:Samtec_HLE-120-02-xx-DV-TE_2x20_P2.54mm_Horizontal -> jrc:JRC_Expansion_Slot
Connections:
- net PHI2 is gone; now on net XPHI2: J9.12 (Φ2)
- net RDB is gone; now on net XRDB: J9.14 (~RD)
- net RWB is gone; now on net XRWB: J9.13 (R/~W)
- net WRB is gone; now on net XWRB: J9.15 (~WR)
Changed lines of the file:
@@
 Wire Wire Line
 	8800 2650 8650 2650
-Text GLabel 8650 2650 0    50   Input ~ 0
-WRB
 Wire Wire Line
 	8800 2550 8650 2550
-Text GLabel 8650 2550 0    50   Input ~ 0
-RDB
 Wire Wire Line
 	10200 3150 10200 3100
@@
 Wire Wire Line
 	8800 2450 8650 2450
-Text GLabel 8650 2450 0    50   Input ~ 0
-RWB
 Wire Wire Line
 	9600 2250 9750 2250
@@
 Wire Wire Line
 	8800 2350 8650 2350
-Text GLabel 8650 2350 0    50   Input ~ 0
-PHI2
 Wire Wire Line
 	9600 2050 9750 2050
@@
 F 0 "J9" H 9200 3500 50  0000 C CNN
 F 1 "SLOT 3" H 9200 3400 50  0000 C CNN
-F 2 "Connector_Samtec_HLE_THT:Samtec_HLE-120-02-xx-DV-TE_2x20_P2.54mm_Horizontal" H 9200 2150 50  0001 C CNN
+F 2 "jrc:JRC_Expansion_Slot" H 9200 2150 50  0001 C CNN
 F 3 "" H 9200 2150 50  0001 C CNN
 	1    9200 2150
@@
 F 0 "J8" H 6750 3500 50  0000 C CNN
 F 1 "SLOT 2" H 6750 3400 50  0000 C CNN
-F 2 "Connector_Samtec_HLE_THT:Samtec_HLE-120-02-xx-DV-TE_2x20_P2.54mm_Horizontal" H 6750 2150 50  0001 C CNN
+F 2 "jrc:JRC_Expansion_Slot" H 6750 2150 50  0001 C CNN
 F 3 "" H 6750 2150 50  0001 C CNN
 	1    6750 2150
@@
 F 0 "J6" H 4350 3500 50  0000 C CNN
 F 1 "SLOT 1" H 4350 3400 50  0000 C CNN
-F 2 "Connector_Samtec_HLE_THT:Samtec_HLE-120-02-xx-DV-TE_2x20_P2.54mm_Horizontal" H 4350 2150 50  0001 C CNN
+F 2 "jrc:JRC_Expansion_Slot" H 4350 2150 50  0001 C CNN
 F 3 "" H 4350 2150 50  0001 C CNN
 	1    4350 2150
@@
 Wire Wire Line
 	9450 5700 9650 5700
+Text GLabel 8650 2650 0    50   Input ~ 0
+XWRB
+Text GLabel 8650 2550 0    50   Input ~ 0
+XRDB
+Text GLabel 8650 2450 0    50   Input ~ 0
+XRWB
+Text GLabel 8650 2350 0    50   Input ~ 0
+XPHI2
 $EndSCHEMATC

Commit message: RC1 of schematic and initial board layout
Parts:
- removed C19, C23, C25: 0.1u, Capacitor_THT:C_Rect_L4.6mm_W2.0mm_P2.50mm_MKS02_FKP02, symbol Device:C_Small
- removed C20, C24, C26: 10u, Capacitor_THT:CP_Radial_D5.0mm_P2.00mm, symbol Device:CP_Small
- added D1: POWER, LED_THT:LED_D5.0mm_Clear, symbol Device:LED
- added H1, H2, H3, H4: MountingHole, MountingHole:MountingHole_2.7mm_M2.5, symbol Mechanical:MountingHole
- added R3: 330, Resistor_THT:R_Axial_DIN0207_L6.3mm_D2.5mm_P10.16mm_Horizontal, symbol Device:R_Small_US
- C19: renamed from C21; footprint Capacitor_THT:CP_Radial_D5.0mm_P2.00mm -> Capacitor_THT:CP_Radial_D6.3mm_P2.50mm
- J1: footprint Connector_PinHeader_1.00mm:PinHeader_2x17_P1.00mm_Vertical -> Connector_PinHeader_2.54mm:PinHeader_2x17_P2.54mm_Vertical
- SW1: value SW_Push -> RESET
- SW2: value SW_Push -> NMI
- renumbered C22 to C20
Connections:
- net +5V: now also D1.2 (A)
- net GND: now also R3.2
- net XA0 renamed A0
- net XA1 renamed A1
- net XA2 renamed A2
- net XA3 renamed A3
- net XA4 renamed A4
- net XA5 renamed A5
- net XA6 renamed A6
- net XA7 renamed A7
- net XD0 renamed D0
- net XD1 renamed D1
- net XD2 renamed D2
- net XD3 renamed D3
- net XD4 renamed D4
- net XD5 renamed D5
- net XD6 renamed D6
- net XD7 renamed D7
- net XPHI2 renamed PHI2
- net XRDB renamed RDB
- net XRWB renamed RWB
- net XWRB renamed WRB
- new net: D1.1 (K), R3.1
Other:
- note added: "Mounting Holes"

Commit message: Fix footprint for RESET and NMI button handlers Fix symbol for '573 latch
Parts:
- U10, U11: footprint jrc:TO-92_reverse -> Package_TO_SOT_THT:TO-92
Changed lines of the file:
@@
 F 0 "U10" H 6600 6000 50  0000 R CNN
 F 1 "DS1813" H 7250 6000 50  0000 R CNN
-F 2 "jrc:TO-92_reverse" H 6800 5650 50  0001 C CNN
+F 2 "Package_TO_SOT_THT:TO-92" H 6800 5650 50  0001 C CNN
 F 3 "" H 6800 5650 50  0001 C CNN
 	1    6800 5650
@@
 F 0 "U11" H 8750 6050 50  0000 R CNN
 F 1 "DS1813" H 9400 6050 50  0000 R CNN
-F 2 "jrc:TO-92_reverse" H 8950 5700 50  0001 C CNN
+F 2 "Package_TO_SOT_THT:TO-92" H 8950 5700 50  0001 C CNN
 F 3 "" H 8950 5700 50  0001 C CNN
 	1    8950 5700
